Commit message: several bugs fixed

File: biorob_bounding_fwd/model/biorob.urdf (robot description, URDF)
Before this commit: robot biorob, 17 links, 16 joints
Links:
- link base: geometry collision mesh filename=./meshes/base.STL; visual mesh filename=meshes/base.STL
- link bl_calf: geometry collision mesh filename=./meshes/BL_calf.STL; visual mesh filename=./meshes/BL_calf.STL
- link bl_foot: geometry collision mesh filename=./meshes/BL_foot.STL; visual mesh filename=./meshes/BL_foot.STL
- link bl_rod: geometry collision mesh filename=./meshes/BL_rod.STL; visual mesh filename=./meshes/BL_rod.STL
- link bl_thigh: geometry collision mesh filename=./meshes/BL_thigh.STL; visual mesh filename=./meshes/BL_thigh.STL
- link br_calf: geometry collision mesh filename=./meshes/BR_calf.STL; visual mesh filename=./meshes/BR_calf.STL
- link br_foot: geometry collision mesh filename=./meshes/BR_foot.STL; visual mesh filename=./meshes/BR_foot.STL
- link br_rod: geometry collision mesh filename=./meshes/BR_rod.STL; visual mesh filename=./meshes/BR_rod.STL
- link br_thigh: geometry collision mesh filename=./meshes/BR_thigh.STL; visual mesh filename=./meshes/BR_thigh.STL
- link fl_calf: geometry collision mesh filename=./meshes/FL_calf.STL; visual mesh filename=./meshes/FL_calf.STL
- link fl_foot: geometry collision mesh filename=./meshes/FL_foot.STL; visual mesh filename=./meshes/FL_foot.STL
- link fl_rod: geometry collision mesh filename=./meshes/FL_rod.STL; visual mesh filename=./meshes/FL_rod.STL
- link fl_thigh: geometry collision mesh filename=./meshes/FL_thigh.STL; visual mesh filename=./meshes/FL_thigh.STL
- link fr_calf: geometry collision mesh filename=./meshes/BR_calf.STL; visual mesh filename=./meshes/BR_calf.STL
- link fr_foot: geometry collision mesh filename=./meshes/FR_foot.STL; visual mesh filename=./meshes/FR_foot.STL
- link fr_rod: geometry collision mesh filename=./meshes/FR_rod.STL; visual mesh filename=./meshes/FR_rod.STL
- link fr_thigh: geometry collision mesh filename=./meshes/FR_thigh.STL; visual mesh filename=./meshes/FR_thigh.STL

File: solo_bounding_fwd/model/solo.urdf (robot description, URDF)
Before this commit: robot solo, 13 links, 12 joints
Links:
- link base: geometry collision mesh filename=./meshes/solo_body.stl; visual mesh filename=./meshes/solo_body.stl
- link bl_foot: geometry collision mesh filename=./meshes/solo_foot.stl; visual mesh filename=./meshes/solo_foot.stl
- link bl_lower_leg: geometry collision mesh filename=./meshes/solo_lower_leg_left_side.stl; visual mesh filename=./meshes/solo_lower_leg_left_side.stl
- link bl_upper_leg: geometry collision mesh filename=./meshes/solo_upper_leg_left_side.stl; visual mesh filename=./meshes/solo_upper_leg_left_side.stl
- link br_foot: geometry collision mesh filename=./meshes/solo_foot.stl; visual mesh filename=./meshes/solo_foot.stl
- link br_lower_leg: geometry collision mesh filename=./meshes/solo_lower_leg_right_side.stl; visual mesh filename=./meshes/solo_lower_leg_right_side.stl
- link br_upper_leg: geometry collision mesh filename=./meshes/solo_upper_leg_right_side.stl; visual mesh filename=./meshes/solo_upper_leg_right_side.stl
- link fl_foot: geometry collision mesh filename=./meshes/solo_foot.stl; visual mesh filename=./meshes/solo_foot.stl
- link fl_lower_leg: geometry collision mesh filename=./meshes/solo_lower_leg_left_side.stl; visual mesh filename=./meshes/solo_lower_leg_left_side.stl
- link fl_upper_leg: geometry collision mesh filename=./meshes/solo_upper_leg_left_side.stl; visual mesh filename=./meshes/solo_upper_leg_left_side.stl
- link fr_foot: geometry collision mesh filename=./meshes/solo_foot.stl; visual mesh filename=./meshes/solo_foot.stl
- link fr_lower_leg: geometry collision mesh filename=./meshes/solo_lower_leg_right_side.stl; visual mesh filename=./meshes/solo_lower_leg_right_side.stl
- link fr_upper_leg: geometry collision mesh filename=./meshes/solo_upper_leg_right_side.stl; visual mesh filename=./meshes/solo_upper_leg_right_side.stl
